Commit message: joint type continuous -> revolute

File: mini_cheetah/mini_cheetah.urdf (robot description, URDF)
Before this commit: robot mini_cheetah, 17 links, 16 joints
Joints:
- joint abduct_fl_to_thigh_fl_j: type continuous -> revolute
- joint abduct_fr_to_thigh_fr_j: type continuous -> revolute
- joint abduct_hl_to_thigh_hl_j: type continuous -> revolute
- joint abduct_hr_to_thigh_hr_j: type continuous -> revolute
- joint thigh_fl_to_knee_fl_j: type continuous -> revolute
- joint thigh_fr_to_knee_fr_j: type continuous -> revolute
- joint thigh_hl_to_knee_hl_j: type continuous -> revolute
- joint thigh_hr_to_knee_hr_j: type continuous -> revolute
- joint torso_to_abduct_fl_j: type continuous -> revolute
- joint torso_to_abduct_fr_j: type continuous -> revolute
- joint torso_to_abduct_hl_j: type continuous -> revolute
- joint torso_to_abduct_hr_j: type continuous -> revolute
